File: pcb/tpms_breakout/tpms_breakout.sch (EAGLE design)
At the start: 21 parts, among them P1 53398-0410, P2 53398-0410, P3 53398-0410, P4 53398-0410, P5 53398-0410, P6 53398-0410, P7 53398-0410, P8 53398-0410, P9 53398-0610

Commit message: initial versions of imu logger, cdh, and tpms pcb
Parts:
- added H1, H2, H3, H4: MOUNT-PAD-ROUND2.8, holes:MOUNT-PAD-ROUND2.8
- renumbered LED1 to PWR, LED2 to ACT, LED3 to RUN, LED4 to ERR, P1 to PS2, P2 to PS5, P3 to PS3, P4 to TC3, P5 to PS1, P6 to TC1, P7 to TC2, P8 to PS4, P9 to CDH
Connections:
- removed net +3V3: JP1.15
- removed net D0: JP1.3
- removed net D1: JP1.2
- removed net D10: JP3.7
- removed net D11: JP3.6
- removed net D12: JP3.5
- removed net D6: JP3.9
- removed net D9: JP3.8
- removed net N$1: CDH.1
- removed net N$10: CDH.6
- removed net N$2: CDH.2
- removed net N$3: CDH.3
- removed net N$4: CDH.4
- removed net N$9: CDH.5
- new net RX1: CDH.4, JP1.3
- new net SCHED: CDH.5, JP3.5
- new net TX1: CDH.3, JP1.2
- net 3V3: now also JP1.15
- net EN: now also CDH.6
- net GND: now also CDH.1, H1.MOUNT, H2.MOUNT, H3.MOUNT, H4.MOUNT
- net LED1: now also JP3.6
- net LED2: now also JP3.7
- net LED3: now also JP3.8
- net LED4: now also JP3.9
- net SC0: now also TC2.2
- net SC1: now also TC3.2
- net SC3: now also PS2.2
- net SC4: now also PS3.2
- net SC5: now also PS4.2
- net SC6: now also PS5.2
- net SC7: now also TC1.2
- net SD0: now also TC2.1
- net SD1: now also TC3.1
- net SD3: now also PS2.1
- net SD4: now also PS3.1
- net SD5: now also PS4.1
- net SD6: now also PS5.1
- net SD7: now also TC1.1
- net VBAT: now also CDH.2

Commit message: finished TPMS board and other updates
Other:
- note added: "Feather M0 Breakout (SAMD21)"
- note added: "Main CDH connector"
- note added: "Mounting holes"
- note added: "Pressure sensor connectors"
- note added: "Status LEDs"
- note added: "TC to digital connectors"
- moved on the sheet: JP1, JP3
