File: pcb/main_board/main_board.brd (EAGLE design)
At the start: 50.8 x 61 mm, 38 parts, among them J1 MEM2067-02-180-00-A_REVB, U13 SPX3819-3.3, U2 SSM6J414TU, U3 SSM6J414TU

Commit message: updated silkscreen and exported cam files for main board
Parts:
- added SJ1: (no value), jumper:SJ
Connections:
- net 9V: now also SJ1.2
- net VBAT: now also SJ1.1
Routing:
- net 9V: track 18.1 -> 27.5 mm, vias 1 -> 3
- net VBAT: track 133.6 -> 139.9 mm, vias 5 -> 7
- net V+_IRIDIUM: track 30.4 -> 28.5 mm
- added copper zone on layer 15, net GND
- added copper zone on layer 2, net GND
Other:
- board text added: "3V3"
- board text added: "GPS voltage select"
- board text added: "Jumper or resistor to bridge pyro source and main battery"
- board text added: "Main command and data handling (CDH) board to be part of the avionics for the flight test article (FTA) being built under the additive manufacturing of thermal protective systems (AMTPS) project in conjunction with NASA and the University of Kentucky. Matt Ruffner, John Schmidt (UK) Mykale Holland, David Blette, Adam Sidor (Johnson Space Center) December 2021"
- board text added: "VBAT"
Changed lines of the file:
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@@
 <layers>
 <layer number="1" name="Top" color="4" fill="1" visible="yes" active="yes"/>
-<layer number="2" name="Route2" color="16" fill="1" visible="no" active="no"/>
+<layer number="2" name="Route2" color="16" fill="1" visible="no" active="yes"/>
 <layer number="3" name="Route3" color="17" fill="1" visible="no" active="no"/>
 <layer number="4" name="Route4" color="18" fill="1" visible="no" active="no"/>
@@
 <layer number="13" name="Route13" color="21" fill="1" visible="no" active="no"/>
 <layer number="14" name="Route14" color="22" fill="1" visible="no" active="no"/>
-<layer number="15" name="Route15" color="23" fill="1" visible="no" active="no"/>
+<layer number="15" name="Route15" color="23" fill="1" visible="no" active="yes"/>
 <layer number="16" name="Bottom" color="1" fill="1" visible="yes" active="yes"/>
 <layer number="17" name="Pads" color="2" fill="1" visible="yes" active="yes"/>
@@
 <wire x1="48.26" y1="60.96" x2="2.54" y2="60.96" width="0" layer="20"/>
 <wire x1="2.54" y1="60.96" x2="0" y2="58.42" width="0" layer="20" curve="90"/>
-<dimension x1="0" y1="-12.7" x2="50.8" y2="-12.7" x3="25.4" y3="-5.08" textsize="1.778" layer="1" unit="inch"/>
-<dimension x1="-12.7" y1="0" x2="-12.7" y2="60.96" x3="-5.08" y3="30.48" textsize="1.778" layer="1" dtype="horizontal" unit="inch"/>
 <text x="48.768" y="6.604" size="1.27" layer="25" font="vector" rot="R90">AMTPS FTA CDH PCB</text>
 <text x="45.085" y="18.415" size="1.016" layer="25" font="vector" rot="R270">Matt Ruffner 2021</text>
@@
 RX
 TX</text>
-<text x="48.895" y="27.432" size="0.8128" layer="26" font="vector" rot="MR0">GND
+<text x="47.244" y="30.48" size="0.8128" layer="26" font="vector" rot="MR0">GND
 VBAT
 RX
@@
 5V
 EN</text>
+<text x="48.895" y="11.303" size="1.016" layer="26" rot="MR0">Main command and data handling (CDH) board
+to be part of the avionics for the flight test article (FTA)  being
+built under the additive manufacturing of thermal protective
+systems (AMTPS) project in conjunction with NASA
+and the University of Kentucky.
+Matt Ruffner, John Schmidt (UK)
+Mykale Holland, David Blette,
+Adam Sidor (Johnson Space Center)
+               December 2021</text>
+<wire x1="48.26" y1="38.1" x2="43.18" y2="38.1" width="0.508" layer="26"/>
+<wire x1="43.18" y1="38.1" x2="43.18" y2="29.845" width="0.508" layer="26"/>
+<wire x1="43.18" y1="29.845" x2="48.26" y2="29.845" width="0.508" layer="26"/>
+<wire x1="48.26" y1="29.845" x2="48.26" y2="38.1" width="0.508" layer="26"/>
+<text x="29.21" y="3.302" size="1.016" layer="26" rot="MR0">GPS voltage
+select</text>
+<text x="24.384" y="6.35" size="1.016" layer="26" rot="MR0">VBAT</text>
+<text x="24.384" y="9.652" size="1.016" layer="26" rot="MR0">3V3</text>
+<text x="31.242" y="53.467" size="1.016" layer="26" rot="MR0">Jumper or resistor to
+bridge pyro source
+and main battery</text>
 </plain>
 <attributes>
@@
 necessary adjustments and save your customized
 design rules under a new name.</description>
-<param name="layerSetup" value="(1*16)"/>
+<param name="layerSetup" value="(1+2*15+16)"/>
 <param name="mtCopper" value="0.035mm 0.035mm 0.035mm 0.035mm 0.035mm 0.035mm 0.035mm 0.035mm 0.035mm 0.035mm 0.035mm 0.035mm 0.035mm 0.035mm 0.035mm 0.035mm"/>
 <param name="mtIsolate" value="1.5mm 0.15mm 0.2mm 0.15mm 0.2mm 0.15mm 0.2mm 0.15mm 0.2mm 0.15mm 0.2mm 0.15mm 0.2mm 0.15mm 0.2mm"/>
@@
 </element>
 <element name="JMP1" library="jump-0r-smd" library_urn="urn:adsk.eagle:library:251" package="A0R-JMP" package3d_urn="urn:adsk.eagle:package:15385/1" value="0R-JUMPA" x="25.527" y="8.509" smashed="yes" rot="MR180">
-<attribute name="NAME" x="24.765" y="5.793" size="1.27" layer="26" rot="MR180"/>
 <attribute name="POPULARITY" value="3" x="25.527" y="8.509" size="1.016" layer="28" rot="MR180" display="off"/>
 <attribute name="VALUE" x="24.765" y="12.495" size="1.27" layer="28" rot="MR180"/>
@@
 <attribute name="SPICEPREFIX" value="C" x="6.223" y="47.371" size="1.016" layer="27" rot="R180" display="off"/>
 <attribute name="VALUE" x="6.858" y="49.276" size="1.27" layer="27" rot="R180"/>
+</element>
+<element name="SJ1" library="jumper" library_urn="urn:adsk.eagle:library:252" package="SJ" package3d_urn="urn:adsk.eagle:package:15471/1" value="" x="24.765" y="51.435" smashed="yes" rot="MR180">
+<attribute name="NAME" x="23.114" y="50.292" size="1.27" layer="26" ratio="10" rot="MR180"/>
+<attribute name="POPULARITY" value="33" x="24.765" y="51.435" size="1.016" layer="28" rot="MR180" display="off"/>
+<attribute name="VALUE" x="25.1651" y="51.435" size="0.02" layer="28" rot="MR180"/>
 </element>
 </elements>
@@
 <wire x1="7.493" y1="41.529" x2="7.62" y2="41.656" width="0.254" layer="16"/>
 <wire x1="7.62" y1="41.656" x2="7.62" y2="41.91" width="0.254" layer="16"/>
+<polygon width="0.254" layer="2">
+<vertex x="-1.27" y="63.5"/>
+<vertex x="54.61" y="63.5"/>
+<vertex x="54.61" y="-2.54"/>
+<vertex x="53.34" y="-3.81"/>
+<vertex x="-1.27" y="-3.81"/>
+<vertex x="-2.54" y="-2.54"/>
+<vertex x="-2.54" y="62.23"/>
+</polygon>
+<polygon width="0.254" layer="15">
+<vertex x="-3.81" y="63.5"/>
+<vertex x="52.07" y="63.5"/>
+<vertex x="52.07" y="-2.54"/>
+<vertex x="50.8" y="-3.81"/>
+<vertex x="-3.81" y="-3.81"/>
+<vertex x="-5.08" y="-2.54"/>
+<vertex x="-5.08" y="62.23"/>
+</polygon>
 </signal>
 <signal name="3V3">
@@
 <wire x1="16.51" y1="41.361" x2="16.51" y2="40.64" width="1.016" layer="1"/>
 <wire x1="19.685" y1="54.737" x2="19.685" y2="53.467" width="0.8128" layer="1"/>
-<wire x1="21.082" y1="52.07" x2="19.685" y2="53.467" width="0.8128" layer="1"/>
-<wire x1="21.082" y1="52.07" x2="21.082" y2="46.695" width="0.8128" layer="1"/>
+<wire x1="19.685" y1="53.467" x2="21.082" y2="52.07" width="0.8128" layer="1"/>
+<wire x1="21.082" y1="46.695" x2="21.082" y2="50.8" width="0.8128" layer="1"/>
 <wire x1="21.082" y1="46.695" x2="20.107" y2="45.72" width="0.8128" layer="1"/>
 <wire x1="20.107" y1="45.72" x2="18.837" y2="45.72" width="0.8128" layer="1"/>
@@
 <wire x1="13.9192" y1="2.0828" x2="25.0698" y2="2.0828" width="0.6096" layer="1"/>
 <wire x1="25.0698" y1="2.0828" x2="27.432" y2="4.445" width="0.6096" layer="1"/>
+<contactref element="SJ1" pad="1"/>
+<via x="21.082" y="50.8" extent="1-16" drill="0.35"/>
+<wire x1="21.082" y1="50.8" x2="23.368" y2="50.8" width="0.8128" layer="16"/>
+<wire x1="23.368" y1="50.8" x2="24.003" y2="51.435" width="0.8128" layer="16"/>
+<wire x1="21.082" y1="52.07" x2="21.082" y2="50.8" width="0.8128" layer="1"/>
+<wire x1="24.003" y1="51.435" x2="23.495" y2="51.943" width="0.8128" layer="16"/>
+<wire x1="23.495" y1="51.943" x2="21.082" y2="51.943" width="0.8128" layer="16"/>
+<via x="21.082" y="52.07" extent="1-16" drill="0.35"/>
 <wire x1="12.507" y1="35.306" x2="13.777" y2="35.306" width="0" layer="19" extent="1-1"/>
 <wire x1="11.237" y1="35.306" x2="12.507" y2="35.306" width="0" layer="19" extent="1-1"/>
@@
 <wire x1="18.288" y1="51.349" x2="18.288" y2="52.197" width="0.8128" layer="1"/>
 <via x="18.288" y="52.197" extent="1-16" drill="0.35"/>
-<wire x1="18.288" y1="52.197" x2="21.463" y2="52.197" width="0.8128" layer="16"/>
-<wire x1="21.463" y1="52.197" x2="22.86" y2="50.8" width="0.8128" layer="16"/>
-<wire x1="22.86" y1="50.8" x2="22.86" y2="46.482" width="0.8128" layer="16"/>
+<wire x1="22.86" y1="46.99" x2="18.288" y2="51.562" width="0.8128" layer="16"/>
+<wire x1="18.288" y1="52.197" x2="18.288" y2="51.562" width="0.8128" layer="16"/>
+<wire x1="22.86" y1="46.99" x2="22.86" y2="46.482" width="0.8128" layer="16"/>
 <via x="19.304" y="52.197" extent="1-16" drill="0.35"/>
 <wire x1="22.86" y1="45.847" x2="22.86" y2="46.482" width="0.8128" layer="16"/>
@@
 <wire x1="35.345" y1="43.18" x2="34.798" y2="43.18" width="0.3048" layer="16"/>
 <wire x1="34.798" y1="43.18" x2="33.909" y2="44.069" width="0.3048" layer="16"/>
+<contactref element="SJ1" pad="2"/>
+<via x="29.972" y="52.07" extent="1-16" drill="0.35"/>
+<via x="29.972" y="50.8" extent="1-16" drill="0.35"/>
+<wire x1="25.527" y1="51.435" x2="26.162" y2="52.07" width="0.8128" layer="16"/>
+<wire x1="26.162" y1="52.07" x2="29.972" y2="52.07" width="0.8128" layer="16"/>
+<wire x1="25.527" y1="51.435" x2="26.162" y2="50.8" width="0.8128" layer="16"/>
+<wire x1="26.162" y1="50.8" x2="29.972" y2="50.8" width="0.8128" layer="16"/>
+<wire x1="30.597" y1="54.737" x2="29.972" y2="52.07" width="0" layer="19" extent="1-1"/>
 </signal>
 <signal name="3V32">
