File: pcb/imu_logger/imu_logger.brd (EAGLE design)
At the start: 50.8 x 22.9 mm, 27 parts, among them J1 DM3CS-SF, P1 53398-0310, U1 MAX14591ETAT, U2 LP2985IM5-1.8/NOPB, U3 MAX14591ETAT, U4 MAX14591ETAT, U5 ICM-20948, U6 ICM-20789

Commit message: initial versions of imu logger, cdh, and tpms pcb
Other:
- board text added: "AMTPS FTA IMU PCB"
- board text removed: "IMU Logger, AMTPS FTA"
Changed lines of the file:
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@@
 <circle x="48.26" y="20.32" radius="1.27" width="0.0254" layer="20"/>
 <circle x="48.26" y="2.54" radius="1.27" width="0.0254" layer="20"/>
-<text x="5.588" y="19.177" size="0.8128" layer="25" font="vector" ratio="9">IMU Logger, AMTPS FTA</text>
+<text x="5.588" y="19.177" size="0.8128" layer="25" font="vector" ratio="9">AMTPS FTA IMU PCB</text>
 <text x="6.604" y="2.667" size="0.8128" layer="25" font="vector" ratio="9">Matt Ruffner, 2021</text>
 <wire x1="44.323" y1="11.557" x2="43.434" y2="11.557" width="0.2032" layer="25"/>

Commit message: add imu board cam files and replace sd card holder
Parts:
- removed J1: DM3CS-SF, DM3CS-SF:HRS_DM3CS-SF
- added J2: MEM2067-02-180-00-A_REVB, MEM20267:GCT_MEM2067-02-180-00-A_REVB
Connections:
- net 3V3: now also J2.4; no longer J1.4
- net GND: now also J2.10, J2.11, J2.12, J2.6, J2.9; no longer J1.6, J1.S1, J1.S2, J1.S3, J1.S5
- net MISO: now also J2.7; no longer J1.7
- net MOSI: now also J2.3; no longer J1.3
- net SCK: now also J2.5; no longer J1.5
- net SD_CS: now also J2.2; no longer J1.2
Routing:
- net SCK: track 18.6 -> 14.7 mm
- net MISO: track 12.4 -> 9.46 mm
- net GND: track 73.3 -> 71.6 mm
- net 3V3: track 35.3 -> 33.8 mm
